Commit message: added HLIP controller wip.

File: models/achilles_SE2_drake.urdf (robot description, URDF)
Before this commit: robot achilles, 32 links, 32 joints
Links:
- added link left_foot
- added link right_foot
Joints:
- added joint left_foot_joint: type fixed, parent left_ankle_pitch, child left_foot, origin xyz=0 0 0 rpy=0 0 0
- added joint right_foot_joint: type fixed, parent right_ankle_pitch, child right_foot, origin xyz=0 0 0 rpy=0 0 0

File: models/achilles_drake.urdf (robot description, URDF)
Before this commit: robot achilles, 31 links, 30 joints
Links:
- added link left_foot
- added link right_foot
Joints:
- added joint left_foot_joint: type fixed, parent left_ankle_pitch, child left_foot, origin xyz=0 0 0 rpy=0 0 0
- added joint right_foot_joint: type fixed, parent right_ankle_pitch, child right_foot, origin xyz=0 0 0 rpy=0 0 0

Commit message: some progress on HLIP. wip

File: models/achilles_SE2_drake.urdf (robot description, URDF)
Before this commit: robot achilles, 34 links, 34 joints
Joints:
- joint left_ankle_pitch_joint: limit lower=-1 upper=1 effort=35 velocity=20 -> (none)
- joint left_elbow_pitch_joint: limit lower=-1.58 upper=0 effort=24 velocity=10 -> (none); type revolute -> fixed
- joint left_hip_pitch_joint: limit lower=-1.5 upper=0.5 effort=35.0 velocity=20 -> (none)
- joint left_hip_roll_joint: limit lower=-1 upper=1 effort=70.0 velocity=10 -> (none)
- joint left_hip_yaw_joint: limit lower=-1 upper=1 effort=35.0 velocity=20 -> (none)
- joint left_knee_pitch_joint: limit lower=0 upper=2 effort=70.0 velocity=10 -> (none)
- joint left_shoulder_pitch_joint: limit lower=-1.58 upper=1.58 effort=35 velocity=20 -> (none); type revolute -> fixed
- joint left_shoulder_roll_joint: limit lower=0 upper=3.141592653589793 effort=12 velocity=20 -> (none)
- joint left_shoulder_yaw_joint: limit lower=-1.58 upper=1.58 effort=12 velocity=20 -> (none)
- joint right_ankle_pitch_joint: limit lower=-1 upper=1 effort=35 velocity=20 -> (none)
- joint right_elbow_pitch_joint: limit lower=-1.58 upper=0 effort=24 velocity=20 -> (none); type revolute -> fixed
- joint right_hip_pitch_joint: limit lower=-1.5 upper=1.5 effort=35.0 velocity=20 -> (none)
- joint right_hip_roll_joint: limit lower=-1 upper=1 effort=70.0 velocity=10 -> (none)
- joint right_hip_yaw_joint: limit lower=-1 upper=1 effort=35.0 velocity=20 -> (none)
- joint right_knee_pitch_joint: limit lower=0 upper=2 effort=70.0 velocity=10 -> (none)
- joint right_shoulder_pitch_joint: limit lower=-1.58 upper=1.58 effort=35 velocity=20 -> (none); type revolute -> fixed
- joint right_shoulder_roll_joint: limit lower=-3.14 upper=0 effort=35 velocity=20 -> (none)
- joint right_shoulder_yaw_joint: limit lower=-1.58 upper=1.58 effort=12.0 velocity=20 -> (none)

File: models/achilles_drake.urdf (robot description, URDF)
Before this commit: robot achilles, 33 links, 32 joints
Joints:
- joint left_hip_pitch_joint: limit lower=-1.5 upper=0.5 effort=35.0 velocity=20 -> lower=-1.5 upper=1.5 effort=35.0 velocity=20

Commit message: got some unstable walking now. wip

File: models/achilles_SE2_drake.urdf (robot description, URDF)
Before this commit: robot achilles, 34 links, 34 joints
Joints:
- joint left_ankle_pitch_joint: limit (none) -> lower=-1 upper=1 effort=35 velocity=20
- joint left_elbow_pitch_joint: limit (none) -> lower=-1.58 upper=0 effort=24 velocity=10
- joint left_hip_pitch_joint: limit (none) -> lower=-1.5 upper=1.5 effort=35.0 velocity=20
- joint left_hip_roll_joint: limit (none) -> lower=-1 upper=1 effort=70.0 velocity=10
- joint left_hip_yaw_joint: limit (none) -> lower=-1 upper=1 effort=35.0 velocity=20
- joint left_knee_pitch_joint: limit (none) -> lower=0 upper=2 effort=70.0 velocity=10
- joint left_shoulder_pitch_joint: limit (none) -> lower=-1.58 upper=1.58 effort=35 velocity=20
- joint left_shoulder_roll_joint: limit (none) -> lower=0 upper=3.141592653589793 effort=12 velocity=20
- joint left_shoulder_yaw_joint: limit (none) -> lower=-1.58 upper=1.58 effort=12 velocity=20
- joint right_ankle_pitch_joint: limit (none) -> lower=-1 upper=1 effort=35 velocity=20
- joint right_elbow_pitch_joint: limit (none) -> lower=-1.58 upper=0 effort=24 velocity=20
- joint right_hip_pitch_joint: limit (none) -> lower=-1.5 upper=1.5 effort=35.0 velocity=20
- joint right_hip_roll_joint: limit (none) -> lower=-1 upper=1 effort=70.0 velocity=10
- joint right_hip_yaw_joint: limit (none) -> lower=-1 upper=1 effort=35.0 velocity=20
- joint right_knee_pitch_joint: limit (none) -> lower=0 upper=2 effort=70.0 velocity=10
- joint right_shoulder_pitch_joint: limit (none) -> lower=-1.58 upper=1.58 effort=35 velocity=20
- joint right_shoulder_roll_joint: limit (none) -> lower=-3.14 upper=0 effort=35 velocity=20
- joint right_shoulder_yaw_joint: limit (none) -> lower=-1.58 upper=1.58 effort=12.0 velocity=20
- joint static_com_joint: origin xyz=0 0 0 rpy=0 0 0 -> xyz=-0.0019 0 -0.286 rpy=0 0 0
