Commit message: almost have 3D walking, just need alittle bit more tuning. wip

File: models/achilles_SE3_drake.urdf (robot description, URDF)
Before this commit: robot achilles, 33 links, 32 joints
Links:
- removed link base
- added link base_link
Joints:
- joint base_to_torso_joint: parent base -> base_link
