Commit message: added 3D IK test

File: models/achilles_SE3_drake_ik.urdf (robot description, URDF)
Before this commit: robot achilles, 34 links, 34 joints
Links:
- removed link base_x
- removed link base_z
- added link base_link
Joints:
- removed joint base_x_joint
- removed joint base_z_joint
- added joint base_to_world_joint: type fixed, parent world, child base_link, origin xyz=0 0 0 rpy=0 0 0
- joint base_to_torso_joint: axis 0 1 0 -> (none); origin xyz=0 0 0 rpy=0 0 0 -> xyz=0 0 1.1 rpy=0 0 0; parent base_z -> base_link
- joint left_hip_roll_joint: type fixed -> revolute
- joint left_hip_yaw_joint: type fixed -> revolute
- joint right_hip_roll_joint: type fixed -> revolute
- joint right_hip_yaw_joint: type fixed -> revolute

Commit message: started HLP control in stance foot frame

File: models/achilles_SE3_drake_ik.urdf (robot description, URDF)
Before this commit: robot achilles, 33 links, 33 joints
Joints:
- joint base_to_torso_joint: origin xyz=0 0 1.1 rpy=0 0 0 -> xyz=0 0 1.1 rpy=0 0 0.78
