Commit message: fixed 2D frontal HLIP once and for all after looking at it with Adrian.

File: models/achilles_SE2_drake_frontal.urdf (robot description, URDF)
Before this commit: robot achilles, 34 links, 34 joints
Joints:
- joint left_hip_yaw_joint: origin xyz=0 0.090 -0.334 rpy=0 0 0 -> xyz=0 0.090 -0.048 rpy=0 0 0
- joint left_shoulder_pitch_joint: origin xyz=0 0.159 0 rpy=0 0 0 -> xyz=0 0.159 0.286 rpy=0 0 0
- joint right_hip_yaw_joint: origin xyz=0 -0.090 -0.334 rpy=0 0 0 -> xyz=0 -0.090 -0.048 rpy=0 0 0
- joint right_shoulder_pitch_joint: origin xyz=0 -0.159 0 rpy=0 0 0 -> xyz=0 -0.159 0.286 rpy=0 0 0
- joint static_com_joint: origin xyz=-0.0019 0 -0.286 rpy=0 0 0 -> xyz=-0.05 0 -0.0 rpy=0 0 0

Commit message: cleaned up 2D frontal walking

File: models/achilles_SE2_drake_frontal.urdf (robot description, URDF)
Before this commit: robot achilles, 34 links, 34 joints
Joints:
- joint left_hip_yaw_joint: origin xyz=0 0.090 -0.048 rpy=0 0 0 -> xyz=0 0.090 -0.334 rpy=0 0 0
- joint left_shoulder_pitch_joint: origin xyz=0 0.159 0.286 rpy=0 0 0 -> xyz=0 0.159 0.0 rpy=0 0 0
- joint right_hip_yaw_joint: origin xyz=0 -0.090 -0.048 rpy=0 0 0 -> xyz=0 -0.090 -0.334 rpy=0 0 0
- joint right_shoulder_pitch_joint: origin xyz=0 -0.159 0.286 rpy=0 0 0 -> xyz=0 -0.159 0.0 rpy=0 0 0
- joint static_com_joint: origin xyz=-0.05 0 -0.0 rpy=0 0 0 -> xyz=-0.0019 0 -0.286 rpy=0 0 0
