Commit message: first attempt at 3D mpc+HLIP with arms.

File: models/achilles_drake.urdf (robot description, URDF)
Before this commit: robot achilles, 33 links, 32 joints
Links:
- link left_hand: geometry collision sphere radius=0.031; visual sphere radius=0.031
- link right_hand: geometry collision sphere radius=0.031; visual sphere radius=0.031
Joints:
- joint left_hand_joint: origin xyz=0.0 0.0 -0.19 rpy=0 0 0 -> xyz=0.0 0.0 -0.192 rpy=0 0 0
- joint right_hand_joint: origin xyz=0.0 0.0 -0.19 rpy=0 0 0 -> xyz=0.0 0.0 -0.192 rpy=0 0 0

Commit message: fixed the torso and com conicedence. They are now offset and do not give IK errors.

File: models/achilles_drake.urdf (robot description, URDF)
Before this commit: robot achilles, 33 links, 32 joints
Joints:
- joint static_com_joint: origin xyz=0 0 0 rpy=0 0 0 -> xyz=-0.0019 0 -0.286 rpy=0 0 0

Commit message: improved standing position based on ZMP-like criterion

File: models/achilles_drake.urdf (robot description, URDF)
Before this commit: robot achilles, 33 links, 32 joints
Joints:
- joint static_com_joint: origin xyz=-0.0019 0 -0.286 rpy=0 0 0 -> xyz=-0.001 0 -0.28 rpy=0 0 0

Commit message: verified the input limit satisfaction from the URDF. Also updated the urdf to have the torque limits from Unitree and Tmotor.

File: models/achilles_drake.urdf (robot description, URDF)
Before this commit: robot achilles, 33 links, 32 joints
Joints:
- joint left_elbow_pitch_joint: limit lower=-1.58 upper=0 effort=24 velocity=10 -> lower=-1.58 upper=0 effort=9 velocity=10
- joint left_hip_roll_joint: limit lower=-1 upper=1 effort=70.0 velocity=10 -> lower=-1 upper=1 effort=35.0 velocity=10
- joint left_shoulder_roll_joint: limit lower=0 upper=3.141592653589793 effort=12 velocity=20 -> lower=0 upper=3.141592653589793 effort=9 velocity=20
- joint left_shoulder_yaw_joint: limit lower=-1.58 upper=1.58 effort=12 velocity=20 -> lower=-1.58 upper=1.58 effort=9 velocity=20
- joint right_elbow_pitch_joint: limit lower=-1.58 upper=0 effort=24 velocity=20 -> lower=-1.58 upper=0 effort=9 velocity=20
- joint right_hip_roll_joint: limit lower=-1 upper=1 effort=70.0 velocity=10 -> lower=-1 upper=1 effort=35.0 velocity=10
- joint right_shoulder_roll_joint: limit lower=-3.14 upper=0 effort=35 velocity=20 -> lower=-3.14 upper=0 effort=9 velocity=20
- joint right_shoulder_yaw_joint: limit lower=-1.58 upper=1.58 effort=12.0 velocity=20 -> lower=-1.58 upper=1.58 effort=9.0 velocity=20

Commit message: added flag for MPC only.

File: models/achilles_drake.urdf (robot description, URDF)
Before this commit: robot achilles, 33 links, 32 joints
Joints:
- joint left_knee_pitch_joint: limit lower=0 upper=2 effort=70.0 velocity=10 -> lower=0 upper=2 effort=35.0 velocity=10
- joint right_knee_pitch_joint: limit lower=0 upper=2 effort=70.0 velocity=10 -> lower=0 upper=2 effort=35.0 velocity=10

Commit message: swapped the torso out for the hardware one

File: models/achilles_drake.urdf (robot description, URDF)
Before this commit: robot achilles, 33 links, 32 joints
Links:
- link torso: geometry visual mesh filename=../meshes/achilles_obj/torso_rough.obj
