Commit message: added actuators to URDF and reduced the contact geometries to the 4 points per foot

File: models/g1_12dof_obj.urdf (robot description, URDF)
Before this commit: robot g1_12dof, 31 links, 30 joints
Links:
- link head_link: geometry visual mesh filename=meshes/head_link.OBJ
- link left_ankle_pitch_link: geometry visual mesh filename=meshes/left_ankle_pitch_link.OBJ
- link left_elbow_link: geometry visual mesh filename=meshes/left_elbow_link.OBJ
- link left_hip_pitch_link: geometry visual mesh filename=meshes/left_hip_pitch_link.OBJ
- link left_hip_roll_link: geometry visual mesh filename=meshes/left_hip_roll_link.OBJ
- link left_hip_yaw_link: geometry visual mesh filename=meshes/left_hip_yaw_link.OBJ
- link left_knee_link: geometry visual mesh filename=meshes/left_knee_link.OBJ
- link left_shoulder_pitch_link: geometry visual mesh filename=meshes/left_shoulder_pitch_link.OBJ
- link left_shoulder_roll_link: geometry visual mesh filename=meshes/left_shoulder_roll_link.OBJ
- link left_shoulder_yaw_link: geometry visual mesh filename=meshes/left_shoulder_yaw_link.OBJ
- link left_wrist_roll_rubber_hand: geometry visual mesh filename=meshes/left_wrist_roll_rubber_hand.OBJ
- link logo_link: geometry visual mesh filename=meshes/logo_link.OBJ
- link pelvis_contour_link: geometry visual mesh filename=meshes/pelvis_contour_link.OBJ
- link right_ankle_pitch_link: geometry visual mesh filename=meshes/right_ankle_pitch_link.OBJ
- link right_elbow_link: geometry visual mesh filename=meshes/right_elbow_link.OBJ
- link right_hip_pitch_link: geometry visual mesh filename=meshes/right_hip_pitch_link.OBJ
- link right_hip_roll_link: geometry visual mesh filename=meshes/right_hip_roll_link.OBJ
- link right_hip_yaw_link: geometry visual mesh filename=meshes/right_hip_yaw_link.OBJ
- link right_knee_link: geometry visual mesh filename=meshes/right_knee_link.OBJ
- link right_shoulder_pitch_link: geometry visual mesh filename=meshes/right_shoulder_pitch_link.OBJ
- link right_shoulder_roll_link: geometry visual mesh filename=meshes/right_shoulder_roll_link.OBJ
- link right_shoulder_yaw_link: geometry visual mesh filename=meshes/right_shoulder_yaw_link.OBJ
- link right_wrist_roll_rubber_hand: geometry visual mesh filename=meshes/right_wrist_roll_rubber_hand.OBJ
- link torso_link: geometry visual mesh filename=meshes/torso_link_23dof_rev_1_0.OBJ
