Commit message: added reference trajecotry for the full order G1 model

File: models/g1_no_hands_obj.urdf (robot description, URDF)
Before this commit: robot g1, 54 links, 53 joints
Links:
- link head_link: geometry visual mesh filename=meshes/head_link.OBJ
- link left_ankle_pitch_link: geometry visual mesh filename=meshes/left_ankle_pitch_link.OBJ
- link left_elbow_link: geometry visual mesh filename=meshes/left_elbow_link.OBJ
- link left_hand_index_0_link: geometry visual mesh filename=meshes/left_hand_index_0_link.OBJ
- link left_hand_index_1_link: geometry visual mesh filename=meshes/left_hand_index_1_link.OBJ
- link left_hand_middle_0_link: geometry visual mesh filename=meshes/left_hand_middle_0_link.OBJ
- link left_hand_middle_1_link: geometry visual mesh filename=meshes/left_hand_middle_1_link.OBJ
- link left_hand_palm_link: geometry visual mesh filename=meshes/left_hand_palm_link.OBJ
- link left_hand_thumb_0_link: geometry visual mesh filename=meshes/left_hand_thumb_0_link.OBJ
- link left_hand_thumb_1_link: geometry visual mesh filename=meshes/left_hand_thumb_1_link.OBJ
- link left_hand_thumb_2_link: geometry visual mesh filename=meshes/left_hand_thumb_2_link.OBJ
- link left_hip_pitch_link: geometry visual mesh filename=meshes/left_hip_pitch_link.OBJ
- link left_hip_roll_link: geometry visual mesh filename=meshes/left_hip_roll_link.OBJ
- link left_hip_yaw_link: geometry visual mesh filename=meshes/left_hip_yaw_link.OBJ
- link left_knee_link: geometry visual mesh filename=meshes/left_knee_link.OBJ
- link left_shoulder_pitch_link: geometry visual mesh filename=meshes/left_shoulder_pitch_link.OBJ
- link left_shoulder_roll_link: geometry visual mesh filename=meshes/left_shoulder_roll_link.OBJ
- link left_shoulder_yaw_link: geometry visual mesh filename=meshes/left_shoulder_yaw_link.OBJ
- link left_wrist_pitch_link: geometry visual mesh filename=meshes/left_wrist_pitch_link.OBJ
- link left_wrist_roll_link: geometry visual mesh filename=meshes/left_wrist_roll_link.OBJ
- link left_wrist_yaw_link: geometry visual mesh filename=meshes/left_wrist_yaw_link.OBJ
- link logo_link: geometry visual mesh filename=meshes/logo_link.OBJ
- link pelvis_contour_link: geometry visual mesh filename=meshes/pelvis_contour_link.OBJ
- link right_ankle_pitch_link: geometry visual mesh filename=meshes/right_ankle_pitch_link.OBJ
- link right_elbow_link: geometry visual mesh filename=meshes/right_elbow_link.OBJ
- link right_hand_index_0_link: geometry visual mesh filename=meshes/right_hand_index_0_link.OBJ
- link right_hand_index_1_link: geometry visual mesh filename=meshes/right_hand_index_1_link.OBJ
- link right_hand_middle_0_link: geometry visual mesh filename=meshes/right_hand_middle_0_link.OBJ
- link right_hand_middle_1_link: geometry visual mesh filename=meshes/right_hand_middle_1_link.OBJ
- link right_hand_palm_link: geometry visual mesh filename=meshes/right_hand_palm_link.OBJ
- link right_hand_thumb_0_link: geometry visual mesh filename=meshes/right_hand_thumb_0_link.OBJ
- link right_hand_thumb_1_link: geometry visual mesh filename=meshes/right_hand_thumb_1_link.OBJ
- link right_hand_thumb_2_link: geometry visual mesh filename=meshes/right_hand_thumb_2_link.OBJ
- link right_hip_pitch_link: geometry visual mesh filename=meshes/right_hip_pitch_link.OBJ
- link right_hip_roll_link: geometry visual mesh filename=meshes/right_hip_roll_link.OBJ
- link right_hip_yaw_link: geometry visual mesh filename=meshes/right_hip_yaw_link.OBJ
- link right_knee_link: geometry visual mesh filename=meshes/right_knee_link.OBJ
- link right_shoulder_pitch_link: geometry visual mesh filename=meshes/right_shoulder_pitch_link.OBJ
- link right_shoulder_roll_link: geometry visual mesh filename=meshes/right_shoulder_roll_link.OBJ
- link right_shoulder_yaw_link: geometry visual mesh filename=meshes/right_shoulder_yaw_link.OBJ
- link right_wrist_pitch_link: geometry visual mesh filename=meshes/right_wrist_pitch_link.OBJ
- link right_wrist_roll_link: geometry visual mesh filename=meshes/right_wrist_roll_link.OBJ
- link right_wrist_yaw_link: geometry visual mesh filename=meshes/right_wrist_yaw_link.OBJ
- link torso_link: geometry visual mesh filename=meshes/torso_link_rev_1_0.OBJ
Joints:
- joint waist_pitch_joint: type revolute -> fixed
- joint waist_roll_joint: type revolute -> fixed
- joint waist_yaw_joint: type revolute -> fixed
