Commit message: added a m4 to the back of g1

File: models/titan_obj.urdf (robot description, URDF)
Before this commit: robot g1, 40 links, 39 joints
Links:
- added link m4_link, mass 5.0
Joints:
- added joint m4_joint: type fixed, parent torso_link, child m4_link, origin xyz=-0.08 0 0.14 rpy=0 0 0

Commit message: tried adding meshes for M4 on the back

File: models/titan_obj.urdf (robot description, URDF)
Before this commit: robot g1, 41 links, 40 joints
Links:
- link m4_link: geometry visual mesh filename=meshes/m4.OBJ

Commit message: added COM projection visualization and added some plotting code for the generated trajectories

File: models/titan_obj.urdf (robot description, URDF)
Before this commit: robot g1, 41 links, 40 joints
Links:
- removed link m4_link
Joints:
- removed joint m4_joint
