Commit message: a bunch of new updates

File: models/g1_29dof_m4_obj.urdf (robot description, URDF)
Before this commit: robot g1_29dof, 40 links, 39 joints
Links:
- added link m4_link, mass 5.0; visual mesh filename=meshes/m4_binary.OBJ
Joints:
- added joint m4_joint: type fixed, parent torso_link, child m4_link, origin xyz=-0.08 0 0.14 rpy=0 0 0
